Commit message: end b term

File: urdf/grace.urdf (robot description, URDF)
Before this commit: robot grace_mobile_manipulator, 43 links, 42 joints
Joints:
- joint joint_4: limit lower=-6.28 upper=6.28 effort=0.26 velocity=3 -> lower=-3.14 upper=3.14 effort=0.26 velocity=3

File: urdf/grace_arm_description.urdf.xacro (robot description, xacro)
@@ -3,5 +3,5 @@
      Commit Version: 1.6.0-4-g7f85cfe  Build Version: 1.6.7995.38578
      For more information, please see http://wiki.ros.org/sw_urdf_exporter -->
-<robot xmlns:xacro="http://www.ros.org/wiki/xacro" name="grace_arm">
+<robot xmlns:xacro="http://www.ros.org/wiki/xacro" name="grace">
     <xacro:macro name="grace_arm" params="parent">
     <link name="arm_link">
@@ -350,5 +350,5 @@
     <gazebo>
         <plugin name="gazebo_ros_control" filename="libgazebo_ros_control.so">
-            <robotNamespace>/grace_arm</robotNamespace>
+            <robotNamespace>/grace</robotNamespace>
         </plugin>
     </gazebo>
