Commit message: demo_gazebo works now independent of turtlebot

File: urdf/grace_arm_description.urdf.xacro (robot description, xacro)
@@ -3,6 +3,6 @@
      Commit Version: 1.6.0-4-g7f85cfe  Build Version: 1.6.7995.38578
      For more information, please see http://wiki.ros.org/sw_urdf_exporter -->
-<robot name="grace_arm">
-    <link name="world"/>
+<robot xmlns:xacro="http://www.ros.org/wiki/xacro" name="grace_arm">
+    <xacro:macro name="grace_arm" params="parent">
     <link name="arm_link">
 <inertial>
@@ -31,5 +31,5 @@
     </link>
         <joint name="arm_joint" type="fixed">
-        <parent link="world" />
+        <parent link="${parent}" />
         <child link="arm_link" />
         <origin xyz="0 0 0" rpy="0 0 0" />
@@ -353,3 +353,4 @@
         </plugin>
     </gazebo>
+</xacro:macro>
 </robot>

Commit message: Updated gripper to work properly in sim

File: urdf/grace_arm_description.urdf.xacro (robot description, xacro)
@@ -266,5 +266,4 @@
         <axis xyz="0 -1 0" />
         <limit lower="0" upper="0.02" effort="100" velocity="3" />
-        <mimic joint="joint_7" multiplier="1" offset="0" />
     </joint>
 <transmission name="trans_joint_1">
