Commit message: end of c term

File: urdf/grace_arm_description.urdf (robot description, URDF)
Before this commit: robot grace, 9 links, 8 joints
Joints:
- joint joint_1: limit lower=-6.28 upper=6.28 effort=2.8 velocity=3 -> lower=-1.85005 upper=1.85005 effort=2.8 velocity=3
- joint joint_2: axis 0 -1 0 -> 0 1 0; limit lower=-2.3 upper=0.1739 effort=2.8 velocity=3 -> lower=-0.314159 upper=2.1 effort=2.8 velocity=3
- joint joint_3: limit lower=-1.3831 upper=1.2 effort=2.8 velocity=3 -> lower=-0.610865 upper=0.7833 effort=2.8 velocity=3
- joint joint_4: limit lower=-6.28 upper=6.28 effort=0.26 velocity=3 -> lower=-3.14 upper=3.14 effort=0.26 velocity=3
- joint joint_5: limit lower=-2 upper=2 effort=100 velocity=3 -> lower=-1.74533 upper=1.74533 effort=100 velocity=3

File: urdf/grace_arm_description.urdf.xacro (robot description, xacro)
@@ -62,5 +62,5 @@
         <child link="link_1" />
         <axis xyz="0 0 -1" />
-        <limit lower="-6.28" upper="6.28" effort="2.8" velocity="3" />
+        <limit lower="-1.85005" upper="1.85005" effort="2.8" velocity="3" />
     </joint>
     <link name="link_2">
@@ -90,6 +90,6 @@
         <parent link="link_1" />
         <child link="link_2" />
-        <axis xyz="0 -1 0" />
-        <limit lower="-2.3" upper="0.1739" effort="2.8" velocity="3" />
+        <axis xyz="0 1 0" />
+        <limit lower="-0.314159" upper="1.570795" effort="2.8" velocity="3" />
     </joint>
     <link name="link_3">
@@ -120,5 +120,5 @@
         <child link="link_3" />
         <axis xyz="0 1 0" />
-        <limit lower="-1.3831" upper="1.2" effort="2.8" velocity="3" />
+        <limit lower="-0.610865" upper="0.7833" effort="2.8" velocity="3" />
     </joint>
     <link name="link_4">
@@ -148,6 +148,6 @@
         <parent link="link_3" />
         <child link="link_4" />
-        <axis xyz="1 0 0" />
-        <limit lower="-6.28" upper="6.28" effort="0.26" velocity="3" />
+        <axis xyz="-1 0 0" />
+        <limit lower="-3.14" upper="3.14" effort="0.26" velocity="3" />
     </joint>
     <link name="link_5">
@@ -177,6 +177,6 @@
         <parent link="link_4" />
         <child link="link_5" />
-        <axis xyz="0 1 0" />
-        <limit lower="-2" upper="2" effort="100" velocity="3" />
+        <axis xyz="0 -1 0" />
+        <limit lower="-1.65806" upper="1.65806" effort="100" velocity="3" />
     </joint>
     <link name="link_6">
