Commit message: Tuned the arm

File: grace_arm_description/urdf/grace_arm_description.urdf (robot description, URDF)
Before this commit: robot grace, 9 links, 8 joints
Joints:
- joint joint_4: limit lower=-3.14 upper=3.14 effort=0.26 velocity=3 -> lower=-3.17 upper=3.0 effort=0.26 velocity=3
- joint joint_5: limit lower=-1.74533 upper=1.74533 effort=100 velocity=3 -> lower=-1.65806279 upper=1.65806279 effort=100 velocity=3
- joint joint_6: limit lower=-6.28 upper=6.28 effort=100 velocity=3 -> lower=-2.321 upper=3.11 effort=100 velocity=3

Commit message: Arm J6 zero was moved, made fake_moveit a class, removed some print statements
Co-authored-by: Alexander Beck <AlexanderBeck0@users.noreply.github.com>

File: grace_arm_description/urdf/grace_arm_description.urdf (robot description, URDF)
Before this commit: robot grace, 9 links, 8 joints
Joints:
- joint joint_6: limit lower=-2.321 upper=3.11 effort=100 velocity=3 -> lower=-0.506 upper=5.694 effort=100 velocity=3
