Commit message: Tuned pure pursuit and offsets for picking and placing
Co-authored-by: Alexander Beck <AlexanderBeck0@users.noreply.github.com>

File: grace_arm_description/urdf/grace_arm_description.urdf.xacro (robot description, xacro)
@@ -178,5 +178,5 @@
         <child link="link_5" />
         <axis xyz="0 -1 0" />
-        <limit lower="-1.65806" upper="1.65806" effort="100" velocity="3" />
+        <limit lower="-1.65806279" upper="1.65806279" effort="100" velocity="3" />
     </joint>
     <link name="link_6">
@@ -207,5 +207,5 @@
         <child link="link_6" />
         <axis xyz="1 0 0" />
-        <limit lower="-6.28" upper="6.28" effort="100" velocity="3" />
+        <limit lower="-0.506" upper="5.694" effort="100" velocity="3" />
     </joint>
     <link name="link_7">
